Commit message: Change Model XACRO files structure - Split XACRO Module files onto sub-modules

File: kamtoa_description/urdf/kamtoa_robot.xacro (robot description, xacro)
@@ -3,228 +3,116 @@
     <!-- Wheel file -->
     <xacro:include filename="$(find kamtoa_description)/urdf/wheel.urdf.xacro" />
-    <!-- Definitions for colors -->
-    <material name="Black">
-        <color rgba="0.0 0.0 0.0 1.0" />
-    </material>
-    <material name="Red">
-        <color rgba="0.8 0.0 0.0 1.0" />
-    </material>
-    <material name="White">
-        <color rgba="1.0 1.0 1.0 1.0" />
-    </material>
-    <material name="Blue">
-        <color rgba="0.0 0.0 0.8 1.0" />
-    </material>
-    <!-- Constants (m-kg-s-radians unit system) -->
-    <property name="M_PI" value="3.1415926535897931" />
-    <property name="M_PI_2" value="1.570796327" />
-    <property name="DEG_TO_RAD" value="0.017453293" />
-    <!-- Robot definitions  -->
-    <property name="base_height" value="0.02" />
-    <property name="base_radius" value="0.15" />
-    <property name="base_mass" value="5.0" /> <!-- in kg-->
-    <property name="caster_f_height" value="0.04" />
-    <property name="caster_f_radius" value="0.025" />
-    <property name="caster_f_mass" value="0.5" /> <!-- in kg-->
-    <property name="caster_b_height" value="0.04" />
-    <property name="caster_b_radius" value="0.025" />
-    <property name="caster_b_mass" value="0.5" /> <!-- in kg-->
-    <!-- Wheels -->
-    <property name="wheel_mass" value="2.5" /> --> <!-- in kg-->
-    <property name="base_x_origin_to_wheel_origin" value="0.25" />
-    <property name="base_y_origin_to_wheel_origin" value="0.3" />
-    <property name="base_z_origin_to_wheel_origin" value="0.0" />
-    <!-- Hokuyo Laser scanner -->
-    <property name="hokuyo_size" value="0.05" />
-    <!-- Macro for calculating inertia of cylinder -->
-    <macro name="cylinder_inertia" params="m r h">
-        <inertia  ixx="${m*(3*r*r+h*h)/12}" ixy = "0" ixz = "0"
-                  iyy="${m*(3*r*r+h*h)/12}" iyz = "0"
-                  izz="${m*r*r/2}" />
-    </macro>
-    <!-- Models goes here @@@@@@@@@@@@@@@@@@@@@@@@@@-->
+    <xacro:include filename="$(find kamtoa_description)/urdf/constant.xacro" />
+    <xacro:include filename="$(find kamtoa_description)/urdf/material.xacro" />
+    <xacro:include filename="$(find kamtoa_description)/urdf/hokuyo.xacro" />
+    <xacro:include filename="$(find kamtoa_description)/urdf/diff_drive_plugin.xacro" />
     <!-- Base_Footprint (ground mark)  -->
-        <link name="base_footprint">
-            <inertial>
-              <mass value="0.0001" />
-              <origin xyz="0 0 0" />
-              <inertia ixx="0.0001" ixy="0.0" ixz="0.0"
-                  iyy="0.0001" iyz="0.0"
-                  izz="0.0001" />
-            </inertial>
-            <visual>
-                <origin xyz="0 0 0" rpy="0 0 0" />
-                <geometry>
-                    <box size="0.001 0.001 0.001" />
-                </geometry>
-            </visual>
-        </link>
-        <joint name="base_footprint_joint" type="fixed">
-            <origin xyz="0 0 ${wheel_radius - base_z_origin_to_wheel_origin}"
-                    rpy="0 0 0" />
-            <parent link="base_footprint"/>
-            <child link="base_link" />
-        </joint>
-        <gazebo reference="base_footprint">
-            <turnGravityOff>false</turnGravityOff>
-        </gazebo>
+    <link name="base_footprint">
+    <inertial>
+        <mass value="0.0001" />
+        <origin xyz="0 0 0" />
+        <inertia ixx="0.0001" ixy="0.0" ixz="0.0" iyy="0.0001" iyz="0.0" izz="0.0001" />
+    </inertial>
+    <visual>
+        <origin xyz="0 0 0" rpy="0 0 0" />
+        <geometry>
+            <box size="0.001 0.001 0.001" />
+        </geometry>
+    </visual>
+    </link>
+    <joint name="base_footprint_joint" type="fixed">
+        <origin xyz="0 0 ${wheel_radius - base_z_origin_to_wheel_origin}" rpy="0 0 0" />
+        <parent link="base_footprint" />
+        <child link="base_link" />
+    </joint>
+    <gazebo reference="base_footprint">
+        <turnGravityOff>false</turnGravityOff>
+    </gazebo>
     <!-- Base_Link (Action body/chassis of the robot) -->
-        <link name="base_link">
-            <inertial>
-                <mass value="${base_mass}" />
-                <origin xyz="0 0 0" />
-                <!--The 3x3 rotational inertia matrix. -->
-                <cylinder_inertia m="${base_mass}"
-                                  r="${base_radius}"
-                                  h="${base_height}" />
-            </inertial>
-            <visual>
-                <origin xyz="0 0 0" rpy="0 0 0" />
-                <geometry>
-                    <cylinder length="${base_height}"
-                              radius="${base_radius}" />
-                </geometry>
-                <material name="White" />
-            </visual>
-            <collision>
-                <origin xyz="0 0 0" rpy="0 0 0 " />
-                <geometry>
-                    <cylinder length="${base_height}"
-                              radius="${base_radius}" />
-                </geometry>
-            </collision>
-        </link>
-        <gazebo reference="base_link">
-            <material>Gazebo/White</material>
-            <turnGravityOff>false</turnGravityOff>
-        </gazebo>
+    <link name="base_link">
+    <inertial>
+        <mass value="${base_mass}" />
+        <origin xyz="0 0 0" />
+        <!--The 3x3 rotational inertia matrix. -->
+        <cylinder_inertia m="${base_mass}" r="${base_radius}" h="${base_height}" />
+    </inertial>
+    <visual>
+        <origin xyz="0 0 0" rpy="0 0 0" />
+        <geometry>
+            <cylinder length="${base_height}" radius="${base_radius}" />
+        </geometry>
+        <material name="White" />
+    </visual>
+    <collision>
+        <origin xyz="0 0 0" rpy="0 0 0 " />
+        <geometry>
+            <cylinder length="${base_height}" radius="${base_radius}" />
+        </geometry>
+    </collision>
+    </link>
+    <gazebo reference="base_link">
+        <material>Gazebo/White</material>
+        <turnGravityOff>false</turnGravityOff>
+    </gazebo>
     <!-- Front Caster wheel  -->
-        <link name="caster_front_link">
-            <visual>
-                <origin xyz="0 0.02 0" rpy="${M_PI/2} 0 0" />
-                <geometry>
-                    <sphere radius="${caster_f_radius}" />
-                </geometry>
-                <material name="Black" />
-            </visual>
-            <collision>
-                <geometry>
-                    <sphere radius="${caster_f_radius}" />
-                </geometry>
-                <origin xyz="0 0.02 0" rpy="${M_PI/2} 0 0" />
-            </collision>
-            <inertial>
-                <mass value="${caster_f_mass}" />
-                <origin xyz="0 0 0" />
-                <inertia ixx="0.001" ixy="0.0" ixz="0.0" iyy="0.001" iyz="0.0" izz="0.001" />
-            </inertial>
-        </link>
-        <joint name="caster_front_joint" type="fixed">
-            <parent link="base_link" />
-            <child link="caster_front_link" />
-            <origin xyz="0.115 0.0 0.007" rpy="${-M_PI/2} 0 0" />
-        </joint>
-        <gazebo reference="caster_front_link">
-            <turnGravityOff>false</turnGravityOff>
-        </gazebo>
+    <link name="caster_front_link">
+    <visual>
+        <origin xyz="0 0.02 0" rpy="${M_PI/2} 0 0" />
+        <geometry>
+            <sphere radius="${caster_f_radius}" />
+        </geometry>
+        <material name="Black" />
+    </visual>
+    <collision>
+        <geometry>
+            <sphere radius="${caster_f_radius}" />
+        </geometry>
+        <origin xyz="0 0.02 0" rpy="${M_PI/2} 0 0" />
+    </collision>
+    <inertial>
+        <mass value="${caster_f_mass}" />
+        <origin xyz="0 0 0" />
+        <inertia ixx="0.001" ixy="0.0" ixz="0.0" iyy="0.001" iyz="0.0" izz="0.001" />
+    </inertial>
+    </link>
+    <joint name="caster_front_joint" type="fixed">
+        <parent link="base_link" />
+        <child link="caster_front_link" />
+        <origin xyz="0.115 0.0 0.007" rpy="${-M_PI/2} 0 0" />
+    </joint>
+    <gazebo reference="caster_front_link">
+        <turnGravityOff>false</turnGravityOff>
+    </gazebo>
     <!-- Back Caster wheel  -->
-        <link name="caster_back_link">
-            <visual>
-                <origin xyz="0.02 0.02 0 " rpy="${M_PI/2} 0 0" />
-                <geometry>
-                    <sphere radius="${caster_b_radius}" />
-                </geometry>
-                <material name="Black" />
-            </visual>
-            <collision>
-                <geometry>
-                    <sphere radius="${caster_b_radius}" />
-                </geometry>
-                <origin xyz="0 0.02 0 " rpy="${M_PI/2} 0 0" />
-            </collision>
-            <inertial>
-                <mass value="${caster_b_mass}" />
-                <origin xyz="0 0 0" />
-                <inertia ixx="0.001" ixy="0.0" ixz="0.0" iyy="0.001" iyz="0.0" izz="0.001" />
-            </inertial>
-            </link>
-            <joint name="caster_back_joint" type="fixed">
-                <parent link="base_link" />
-                <child link="caster_back_link" />
-                <origin xyz="-0.135 0.0 0.009" rpy="${-M_PI/2} 0 0" />
-            </joint>
-            <gazebo reference="caster_back_link">
-                <turnGravityOff>false</turnGravityOff>
-            </gazebo>
+    <link name="caster_back_link">
+    <visual>
+        <origin xyz="0.02 0.02 0 " rpy="${M_PI/2} 0 0" />
+        <geometry>
+            <sphere radius="${caster_b_radius}" />
+        </geometry>
+        <material name="Black" />
+    </visual>
+    <collision>
+        <geometry>
+            <sphere radius="${caster_b_radius}" />
+        </geometry>
+        <origin xyz="0 0.02 0 " rpy="${M_PI/2} 0 0" />
+    </collision>
+    <inertial>
+        <mass value="${caster_b_mass}" />
+        <origin xyz="0 0 0" />
+        <inertia ixx="0.001" ixy="0.0" ixz="0.0" iyy="0.001" iyz="0.0" izz="0.001" />
+    </inertial>
+    </link>
+    <joint name="caster_back_joint" type="fixed">
+        <parent link="base_link" />
+        <child link="caster_back_link" />
+        <origin xyz="-0.135 0.0 0.009" rpy="${-M_PI/2} 0 0" />
+    </joint>
+    <gazebo reference="caster_back_link">
+        <turnGravityOff>false</turnGravityOff>
+    </gazebo>
     <!-- Wheel -->
-          <wheel fb="front" lr="right"
-          parent="base_link" translateX="0" translateY="0.5" flipY="1"/>
-          <wheel fb="front" lr="left"
-          parent="base_link" translateX="0" translateY="-0.5" flipY="1"/>
-    <!-- Hokuyo Sensors Model -->
-        <link name="hokuyo_link">
-        <visual>
-            <origin xyz="0 0 0" rpy="0 0 0" />
-            <geometry>
-                <box size="${hokuyo_size} ${hokuyo_size} ${hokuyo_size}" />
-            </geometry>
-            <material name="Blue" />
-        </visual>
-        </link>
-        <joint name="hokuyo_joint" type="fixed">
-            <origin xyz="${base_radius - hokuyo_size/2} 0 ${base_height+hokuyo_size/4}" rpy="0 0 0" />
-            <parent link="base_link" />
-            <child link="hokuyo_link" />
-        </joint>
-        <gazebo reference="hokuyo_link">
-            <material>Gazebo/Blue</material>
-            <turnGravityOff>false</turnGravityOff>
-            <sensor type="ray" name="head_hokuyo_sensor">
-                <pose>${hokuyo_size/2} 0 0 0 0 0</pose>
-                <visualize>false</visualize>
-                <update_rate>40</update_rate>
-                <ray>
-                    <scan>
-                        <horizontal>
-                            <samples>720</samples>
-                            <resolution>1</resolution>
-                            <min_angle>-1.570796</min_angle>
-                            <max_angle>1.570796</max_angle>
-                        </horizontal>
-                    </scan>
-                    <range>
-                        <min>0.10</min>
-                        <max>10.0</max>
-                        <resolution>0.001</resolution>
-                    </range>
-                </ray>
-                <plugin name="gazebo_ros_head_hokuyo_controller" filename="libgazebo_ros_laser.so">
-                    <topicName>/scan</topicName>
-                    <frameName>hokuyo_link</frameName>
-                </plugin>
-            </sensor>
-        </gazebo>
-    <!-- Differential drive controller  -->
-    <gazebo>
-      <plugin name="differential_drive_controller" filename="libgazebo_ros_diff_drive.so">
-        <rosDebugLevel>Debug</rosDebugLevel>
-        <publishWheelTF>false</publishWheelTF>
-        <robotNamespace>/</robotNamespace>
-        <publishTf>1</publishTf>
-        <publishWheelJointState>false</publishWheelJointState>
-        <alwaysOn>true</alwaysOn>
-        <updateRate>100.0</updateRate>
-        <leftJoint>front_left_wheel_joint</leftJoint>
-        <rightJoint>front_right_wheel_joint</rightJoint>
-        <wheelSeparation>${2*base_radius}</wheelSeparation>
-        <wheelDiameter>${2*wheel_radius}</wheelDiameter>
-        <broadcastTF>1</broadcastTF>
-        <wheelTorque>30</wheelTorque>
-        <wheelAcceleration>1.8</wheelAcceleration>
-        <commandTopic>kamtoa/cmd_vel</commandTopic>
-        <odometryFrame>odom</odometryFrame>
-        <odometryTopic>odom</odometryTopic>
-        <robotBaseFrame>base_footprint</robotBaseFrame>
-      </plugin>
-    </gazebo>
+    <wheel fb="front" lr="right" parent="base_link" translateX="0" translateY="0.5" flipY="1" />
+    <wheel fb="front" lr="left" parent="base_link" translateX="0" translateY="-0.5" flipY="1" />
 </robot>

File: kamtoa_description/urdf/wheel.urdf.xacro (robot description, xacro)
@@ -2,15 +2,15 @@
 <robot name="wheel" xmlns:xacro="http://www.ros.org/wiki/xacro">
   <!-- Wheels -->
-  <property name="wheel_radius" value="0.04" />
-  <property name="wheel_height" value="0.02" />
-  <property name="wheel_mass" value="2.5" /> <!-- in kg-->
-  <property name="base_x_origin_to_wheel_origin" value="0.25" />
-  <property name="base_y_origin_to_wheel_origin" value="0.3" />
-  <property name="base_z_origin_to_wheel_origin" value="0.0" />
-  <macro name="cylinder_inertia" params="m r h">
+  <xacro:property name="wheel_radius" value="0.04" />
+  <xacro:property name="wheel_height" value="0.02" />
+  <xacro:property name="wheel_mass" value="2.5" /> <!-- in kg-->
+  <xacro:property name="base_x_origin_to_wheel_origin" value="0.25" />
+  <xacro:property name="base_y_origin_to_wheel_origin" value="0.3" />
+  <xacro:property name="base_z_origin_to_wheel_origin" value="0.0" />
+  <xacro:macro name="cylinder_inertia" params="m r h">
     <inertia  ixx="${m*(3*r*r+h*h)/12}" ixy = "0" ixz = "0"
               iyy="${m*(3*r*r+h*h)/12}" iyz = "0"
               izz="${m*r*r/2}" />
-  </macro>
+  </xacro:macro>
   <xacro:macro name="wheel" params="fb lr parent translateX translateY flipY"> <!--fb : front, back ; lr: left, right -->
     <link name="${fb}_${lr}_wheel">
