Commit message: Add Camera Plugin - Joystick Params for deadman button is set to button 6 - Trigger Value of deadman changed from -1 to 1(support button)

File: kamtoa_description/urdf/constant.xacro (robot description, xacro)
@@ -27,4 +27,7 @@
     <!-- Hokuyo Laser scanner -->
     <xacro:property name="hokuyo_size" value="0.05"/>
+    <!-- Camera Properties -->
+    <xacro:property name="cameraSize" value="0.05"/>
+    <xacro:property name="cameraMass" value="0.1"/>
     <!-- Macro for calculating inertia of cylinder -->
     <xacro:macro name="cylinder_inertia" params="m r h">

File: kamtoa_description/urdf/kamtoa_robot.xacro (robot description, xacro)
@@ -6,4 +6,5 @@
     <xacro:include filename="$(find kamtoa_description)/urdf/material.xacro" />
     <xacro:include filename="$(find kamtoa_description)/urdf/hokuyo.xacro" />
+    <xacro:include filename="$(find kamtoa_description)/urdf/camera.xacro" />
     <xacro:include filename="$(find kamtoa_description)/urdf/diff_drive_plugin.xacro" />
     <!-- Base_Footprint (ground mark)  -->

Commit message: Modified some params in simulation

File: kamtoa_description/urdf/constant.xacro (robot description, xacro)
@@ -11,9 +11,9 @@
     <!-- in kg-->
     <xacro:property name="caster_f_height" value="0.04"/>
-    <xacro:property name="caster_f_radius" value="0.025"/>
+    <xacro:property name="caster_f_radius" value="0.03"/>
     <xacro:property name="caster_f_mass" value="0.5"/>
     <!-- in kg-->
     <xacro:property name="caster_b_height" value="0.04"/>
-    <xacro:property name="caster_b_radius" value="0.025"/>
+    <xacro:property name="caster_b_radius" value="0.027"/>
     <xacro:property name="caster_b_mass" value="0.5"/>
     <!-- in kg-->

File: kamtoa_description/urdf/diff_drive_plugin.xacro (robot description, xacro)
@@ -18,8 +18,8 @@
             <wheelTorque>30</wheelTorque>
             <wheelAcceleration>1.8</wheelAcceleration>
-            <commandTopic>kamtoa/cmd_vel</commandTopic>
+            <commandTopic>cmd_vel</commandTopic>
             <odometryFrame>odom</odometryFrame>
-            <odometryTopic>kamtoa/odom</odometryTopic>
-            <robotBaseFrame>kamtoa/base_footprint</robotBaseFrame>
+            <odometryTopic>odom</odometryTopic>
+            <robotBaseFrame>base_footprint</robotBaseFrame>
             <legacyMode>true</legacyMode> <!-- LegacyMode = true : NORMAL Z Axis : Direcion Up -->
             <odometrySource>1</odometrySource>

File: kamtoa_description/urdf/hokuyo.xacro (robot description, xacro)
@@ -30,8 +30,8 @@
                         <!-- <samples>720</samples> -->
                         <resolution>1</resolution>
-                        <!-- <min_angle>-1.570796</min_angle>
-                        <max_angle>1.570796</max_angle> -->
-                        <min_angle>-3.14</min_angle>
-                        <max_angle>3.14</max_angle>
+                        <!-- --><min_angle>-2</min_angle>
+                        <max_angle>2</max_angle>
+                        <!-- <min_angle>-3.141592</min_angle> -->
+                        <!-- <max_angle>3.141592</max_angle> -->
                     </horizontal>
                 </scan>
@@ -39,8 +39,13 @@
                     <!-- <min>0.10</min>
                     <max>10.0</max> -->
-                    <min>0.15</min>
+                    <min>0.10</min>
                     <max>6</max>
                     <resolution>0.001</resolution>
                 </range>
+                <noise>
+                  <type>gaussian</type>
+                  <mean>0.01</mean>
+                  <stddev>0.015</stddev>
+                </noise>
             </ray>
             <plugin name="gazebo_ros_head_hokuyo_controller" filename="libgazebo_ros_laser.so">

File: kamtoa_description/urdf/kamtoa_robot.xacro (robot description, xacro)
@@ -70,4 +70,14 @@
         </geometry>
         <origin xyz="0 0.02 0" rpy="${M_PI/2} 0 0" />
+        <surface>
+              <friction>
+                <ode>
+                  <mu>0</mu>
+                  <mu2>0</mu2>
+                  <slip1>1.0</slip1>
+                  <slip2>1.0</slip2>
+                </ode>
+              </friction>
+        </surface>
     </collision>
     <inertial>
@@ -99,4 +109,14 @@
         </geometry>
         <origin xyz="0 0.02 0 " rpy="${M_PI/2} 0 0" />
+        <surface>
+              <friction>
+                <ode>
+                  <mu>0</mu>
+                  <mu2>0</mu2>
+                  <slip1>1.0</slip1>
+                  <slip2>1.0</slip2>
+                </ode>
+              </friction>
+        </surface>
     </collision>
     <inertial>

File: kamtoa_description/urdf/wheel.urdf.xacro (robot description, xacro)
@@ -2,5 +2,5 @@
 <robot name="wheel" xmlns:xacro="http://www.ros.org/wiki/xacro">
   <!-- Wheels -->
-  <xacro:property name="wheel_radius" value="0.04" />
+  <xacro:property name="wheel_radius" value="0.041" />
   <xacro:property name="wheel_height" value="0.02" />
   <xacro:property name="wheel_mass" value="2.5" /> <!-- in kg-->
