Commit message: Add Obodroid V10 Model - Integrated the origin of the model - TODO: Add Wheel Plugin , Camera plugin . Laser Plugin

File: som_o_description/urdf/30cm/base_footprint.xacro (robot description, xacro)
@@ -16,8 +16,8 @@
     </link>
     <joint name="base_footprint_joint" type="fixed">
-        <origin xyz="0 0 0" rpy="0 0 0" />
+        <origin xyz="0 0 -${wheel_radius}" rpy="0 0 0" />
         <parent link="base_footprint" />
         <child link="base_link" />
-    </joint>
+    </joint>d
     <gazebo reference="base_footprint">
         <turnGravityOff>false</turnGravityOff>

File: som_o_description/urdf/30cm/base_link.xacro (robot description, xacro)
@@ -9,15 +9,15 @@
       <cylinder_inertia m="${base_mass}" r="${base_radius}" h="${base_height}" />
   </inertial>
-  <!-- [TODO: Create the Mesh from Fusion without wheel and use as ] -->
+  <!-- Base_Link Visual (mesh from STL) -->
   <visual>
-      <origin xyz="0 0 0.055" rpy="0 0 0" />
+      <origin xyz="0 0 0" rpy="0 0 0" />
       <geometry>
-          <mesh filename="package://som_o_description/meshes/full_export.stl"/>
+          <mesh filename="package://som_o_description/meshes/obodroid1.stl"/>
       </geometry>
       <material name="White" />
   </visual>
-  <!-- [TODO : Use BOX Collision Model and except the wheel boundary] -->
+  <!-- Base_Link Collision Model -->
   <collision>
-      <origin xyz="0 0 0" rpy="0 0 0 " />
+      <origin xyz="0 0 ${base_col_box_height/2}" rpy="0 0 0 " />
       <geometry>
           <box size="${base_col_box_length} ${base_col_box_width} ${base_col_box_height}" />

File: som_o_description/urdf/30cm/constants.xacro (robot description, xacro)
@@ -5,21 +5,26 @@
     <xacro:property name="M_PI_2" value="1.570796327"/>
     <xacro:property name="DEG_TO_RAD" value="0.017453293"/>
-    <xacro:property name="thickness" value="0.003"/>
-    <xacro:property name="wheel_radius" value="0.040"/>
     <!-- Base Link Constants -->
     <!-- Inertial components , Mass (Kgs) -->
-    <xacro:property name="base_mass" value="0.040"/>
-    <xacro:property name="base_radius" value="0.400"/>
-    <xacro:property name="base_height" value="0.400"/>
-    <!-- Collision model -->
+    <xacro:property name="base_mass" value="0.2"/>
+    <xacro:property name="base_radius" value="0.20"/>
+    <xacro:property name="base_height" value="0.40"/>
+    <xacro:property name="base_link_visual_mesh_offset_z" value="0.55"/>
+    <!-- Collision 133.091 Origin to base Link model -->
     <!-- Chassis Collsion -->
-    <xacro:property name="base_col_box_height" value="0.250"/>
+    <xacro:property name="base_col_box_height" value="0.300"/>
     <xacro:property name="base_col_box_length" value="0.200"/>
     <xacro:property name="base_col_box_width" value="0.140"/>
-    <!-- <xacro:property name="base_radius" value="0.400"/>
-    <xacro:property name="base_height" value="0.400"/> -->
+    <!-- Wheels -->
+    <xacro:property name="wheel_radius" value="0.042" />
+    <xacro:property name="wheel_height" value="0.026" />
+    <xacro:property name="wheel_mass" value="2.5" /> <!-- in kg-->
+    <xacro:property name="base_x_origin_to_wheel_origin" value="0" />
+    <xacro:property name="base_y_origin_to_wheel_origin" value="0.092" />
+    <xacro:property name="base_z_origin_to_wheel_origin" value="0.00" />
     <!-- Macro for calculating inertia of cylinder -->
     <xacro:macro name="cylinder_inertia" params="m r h">
-        <inertia ixx="${m*(3*r*r+h*h)/12}" ixy="0" ixz="0" iyy="${m*(3*r*r+h*h)/12}" iyz="0" izz="${m*r*r/2}"/>
+        <inertia ixx="${m*(3*r*r+h*h)/12}" ixy="0" ixz="0"
+          iyy="${m*(3*r*r+h*h)/12}" iyz="0" izz="${m*r*r/2}"/>
     </xacro:macro>
 </robot>

File: som_o_description/urdf/30cm/robot_30cm.xacro (robot description, xacro)
@@ -9,3 +9,6 @@
   <xacro:include filename="$(find som_o_description)/urdf/30cm/base_link.xacro" />
   <!-- Wheels (Plugin) -->
+  <xacro:include filename="$(find som_o_description)/urdf/shared_components/wheel.xacro" />
+  <wheel fb="front" lr="right" parent="base_footprint" translateX="0" translateY="1" flipY="1" />
+  <wheel fb="front" lr="left" parent="base_footprint" translateX="0" translateY="-1" flipY="1" />
 </robot>

File: som_o_description/urdf/shared_components/wheel.xacro (robot description, xacro)
@@ -1,16 +1,51 @@
 <?xml version="1.0"?>
 <robot name="wheel" xmlns:xacro="http://www.ros.org/wiki/xacro">
-  <!-- Wheels properties-->
-  <xacro:property name="wheel_radius" value="0.041" />
-  <xacro:property name="wheel_height" value="0.02" />
-  <xacro:property name="wheel_mass" value="2.5" /> <!-- in kg-->
-  <xacro:property name="base_x_origin_to_wheel_origin" value="0.25" />
-  <xacro:property name="base_y_origin_to_wheel_origin" value="0.3" />
-  <xacro:property name="base_z_origin_to_wheel_origin" value="0.0" />
-  <!-- Wheels Inertia calculation macro  -->
-  <xacro:macro name="cylinder_inertia" params="m r h">
-    <inertia  ixx="${m*(3*r*r+h*h)/12}" ixy = "0" ixz = "0"
-              iyy="${m*(3*r*r+h*h)/12}" iyz = "0"
-              izz="${m*r*r/2}" />
-  </xacro:macro>
+<xacro:macro name="wheel" params="fb lr parent translateX translateY flipY"> <!--fb : front, back ; lr: left, right -->
+  <link name="${fb}_${lr}_wheel">
+    <visual>
+      <origin xyz="0 0 0" rpy="${flipY*M_PI/2} 0  0 " />
+      <geometry>
+        <cylinder length="${wheel_height}" radius="${wheel_radius}" />
+      </geometry>
+      <material name="DarkGray" />
+    </visual>
+    <collision>
+      <origin xyz="0 0 0" rpy="${flipY*M_PI/2} 0 0 " />
+      <geometry>
+        <cylinder length="${wheel_height}" radius="${wheel_radius}" />
+      </geometry>
+    </collision>
+    <inertial>
+      <mass value="${wheel_mass}" />
+      <origin xyz="0 0 0" />
+      <cylinder_inertia  m="${wheel_mass}" r="${wheel_radius}" h="${wheel_height}" />
+    </inertial>
+  </link>
+  <gazebo reference="${fb}_${lr}_wheel">
+    <mu1 value="1.0"/>
+    <mu2 value="1.0"/>
+    <kp  value="10000000.0" />
+    <kd  value="1.0" />
+    <fdir1 value="1 0 0"/>
+    <material>Gazebo/Grey</material>
+    <turnGravityOff>false</turnGravityOff>
+  </gazebo>
+  <joint name="${fb}_${lr}_wheel_joint" type="continuous">
+    <parent link="${parent}"/>
+    <child link="${fb}_${lr}_wheel"/>
+    <origin xyz="${translateX * base_x_origin_to_wheel_origin} ${translateY * base_y_origin_to_wheel_origin} ${base_z_origin_to_wheel_origin}" rpy="0 0 0" />
+    <axis xyz="0 1 0" rpy="0  0" />
+    <limit effort="100" velocity="100"/>
+    <joint_properties damping="0.0" friction="0.0"/>
+  </joint>
+  <!-- Transmission is important to link the joints and the controller -->
+  <transmission name="${fb}_${lr}_wheel_joint_trans">
+    <type>transmission_interface/SimpleTransmission</type>
+    <joint name="${fb}_${lr}_wheel_joint" />
+    <actuator name="${fb}_${lr}_wheel_joint_motor">
+      <hardwareInterface>EffortJointInterface</hardwareInterface>
+      <mechanicalReduction>1</mechanicalReduction>
+    </actuator>
+  </transmission>
+</xacro:macro>
 </robot>
