Commit message: Renew file structure of som_o robot - Correct the file name according to its size - Now Model can be spawn by editing just only one argument - TODO: Add Sensors to som_o robot

File: som_o_description/urdf/20cm/base_footprint.xacro (robot description, xacro)
@@ -1,4 +1,4 @@
 <?xml version="1.0"?>
-<robot name="som_o_robot_30cm" xmlns:xacro="http://www.ros.org/wiki/xacro">
+<robot name="som_o_robot_20cm" xmlns:xacro="http://www.ros.org/wiki/xacro">
     <!-- Base_Footprint (ground mark)  -->
     <link name="base_footprint">

File: som_o_description/urdf/20cm/base_link.xacro (robot description, xacro)
@@ -1,4 +1,4 @@
 <?xml version="1.0"?>
-<robot name="som_o_robot_30cm" xmlns:xacro="http://www.ros.org/wiki/xacro">
+<robot name="som_o_robot_20cm" xmlns:xacro="http://www.ros.org/wiki/xacro">
   <!-- Base_Link (Action body/chassis of the robot) -->
   <link name="base_link">

File: som_o_description/urdf/20cm/constants.xacro (robot description, xacro)
@@ -1,17 +1,18 @@
 <?xml version="1.0"?>
-<robot name="som_o_robot_30cm" xmlns:xacro="http://www.ros.org/wiki/xacro">
+<robot name="som_o_robot_20cm" xmlns:xacro="http://www.ros.org/wiki/xacro">
     <!-- Constants (m-kg-s-radians unit system) -->
     <xacro:property name="M_PI" value="3.1415926535897931"/>
     <xacro:property name="M_PI_2" value="1.570796327"/>
     <xacro:property name="DEG_TO_RAD" value="0.017453293"/>
+    <!-- Meterials properties -->
+    <xacro:property name="metal_sheet_thickness" value="0.03"/>
     <!-- Base Link Constants -->
     <!-- Inertial components , Mass (Kgs) -->
     <xacro:property name="base_mass" value="0.2"/>
     <xacro:property name="base_radius" value="0.20"/>
-    <xacro:property name="base_height" value="0.40"/>
+    <xacro:property name="base_height" value="0.22"/>
     <xacro:property name="base_link_visual_mesh_offset_z" value="0.55"/>
-    <!-- Collision 133.091 Origin to base Link model -->
     <!-- Chassis Collsion -->
-    <xacro:property name="base_col_box_height" value="0.300"/>
+    <xacro:property name="base_col_box_height" value="0.183091"/>
     <xacro:property name="base_col_box_length" value="0.200"/>
     <xacro:property name="base_col_box_width" value="0.140"/>

File: som_o_description/urdf/20cm/material.xacro (robot description, xacro)
@@ -1,5 +1,5 @@
 <?xml version="1.0"?>
-<robot name="kamtoa_robot" xmlns:xacro="http://www.ros.org/wiki/xacro">
-<!-- Definitions for colors -->
+<robot name="som_o_robot_20cm" xmlns:xacro="http://www.ros.org/wiki/xacro">
+<!-- Definitions for colors for using in Gazebo and RViz -->
     <material name="Black">
         <color rgba="0.0 0.0 0.0 1.0" />
