Commit message: Add 25,30 Cm Model - More Modular File Structure - Spawning by arguments in param - ex. roslaunch gazebo_som_o.launch size:="30" - More Reusable Component - IMU Added - Multicamera Added

File: som_o_description/urdf/25cm/base_footprint.xacro (robot description, xacro)
@@ -6,5 +6,5 @@
     Author : Theppasith N. <theppasith@gmail.com>
 -->
-<robot name="som_o_robot_20cm" xmlns:xacro="http://www.ros.org/wiki/xacro">
+<robot name="som_o_robot_25cm" xmlns:xacro="http://www.ros.org/wiki/xacro">
     <!-- Base_Footprint (ground mark)  -->
     <link name="base_footprint">

File: som_o_description/urdf/25cm/base_link.xacro (robot description, xacro)
@@ -6,5 +6,5 @@
     Author : Theppasith N. <theppasith@gmail.com>
 -->
-<robot name="som_o_robot_20cm" xmlns:xacro="http://www.ros.org/wiki/xacro">
+<robot name="som_o_robot_25cm" xmlns:xacro="http://www.ros.org/wiki/xacro">
   <!-- Base_Link (Action body/chassis of the robot) -->
   <link name="base_link">

File: som_o_description/urdf/25cm/constants.xacro (robot description, xacro)
@@ -5,5 +5,5 @@
     Author : Theppasith N. <theppasith@gmail.com>
 -->
-<robot name="som_o_robot_20cm" xmlns:xacro="http://www.ros.org/wiki/xacro">
+<robot name="som_o_robot_25cm" xmlns:xacro="http://www.ros.org/wiki/xacro">
     <!-- Constants (m-kg-s-radians unit system) -->
     <xacro:property name="M_PI" value="3.1415926535897931"/>
@@ -15,5 +15,5 @@
     <!-- Inertial components , Mass (kgs) -->
     <xacro:property name="base_mass" value="0.2"/>
-    <xacro:property name="base_radius" value="0.20"/>
+    <xacro:property name="base_radius" value="0.25"/>
     <xacro:property name="base_height" value="0.22"/>
     <xacro:property name="base_link_visual_mesh_offset_z" value="0.55"/>
@@ -21,5 +21,5 @@
     <xacro:property name="base_col_box_height" value="0.183091"/>
     <xacro:property name="base_col_box_length" value="0.200"/>
-    <xacro:property name="base_col_box_width" value="0.130"/>
+    <xacro:property name="base_col_box_width" value="0.180"/>
     <!-- Wheels -->
     <xacro:property name="wheel_radius" value="0.042" />

File: som_o_description/urdf/25cm/som_o_robot_25cm.xacro (robot description, xacro)
@@ -5,14 +5,14 @@
     Author : Theppasith N. <theppasith@gmail.com>
 -->
-<robot name="som_o_robot_20cm" xmlns:xacro="http://www.ros.org/wiki/xacro">
+<robot name="som_o_robot_25cm" xmlns:xacro="http://www.ros.org/wiki/xacro">
   <!-- Constants -->
-  <xacro:include filename="$(find som_o_description)/urdf/20cm/constants.xacro" />
+  <xacro:include filename="$(find som_o_description)/urdf/25cm/constants.xacro" />
   <!-- Material (Color) -->
   <xacro:include filename="$(find som_o_description)/urdf/shared_components/material.xacro" />
   <!-- Body of Robot -->
       <!-- Footprint (require Base Link inclusion) -->
-      <xacro:include filename="$(find som_o_description)/urdf/20cm/base_footprint.xacro" />
+      <xacro:include filename="$(find som_o_description)/urdf/25cm/base_footprint.xacro" />
       <!-- Base Link (Main chassis) -->
-      <xacro:include filename="$(find som_o_description)/urdf/20cm/base_link.xacro" />
+      <xacro:include filename="$(find som_o_description)/urdf/25cm/base_link.xacro" />
       <!-- Wheels (Plugin) -->
       <xacro:include filename="$(find som_o_description)/urdf/shared_components/wheel.xacro" />

File: som_o_description/urdf/30cm/base_footprint.xacro (robot description, xacro)
@@ -6,5 +6,5 @@
     Author : Theppasith N. <theppasith@gmail.com>
 -->
-<robot name="som_o_robot_20cm" xmlns:xacro="http://www.ros.org/wiki/xacro">
+<robot name="som_o_robot_30cm" xmlns:xacro="http://www.ros.org/wiki/xacro">
     <!-- Base_Footprint (ground mark)  -->
     <link name="base_footprint">

File: som_o_description/urdf/30cm/base_link.xacro (robot description, xacro)
@@ -6,5 +6,5 @@
     Author : Theppasith N. <theppasith@gmail.com>
 -->
-<robot name="som_o_robot_20cm" xmlns:xacro="http://www.ros.org/wiki/xacro">
+<robot name="som_o_robot_30cm" xmlns:xacro="http://www.ros.org/wiki/xacro">
   <!-- Base_Link (Action body/chassis of the robot) -->
   <link name="base_link">

File: som_o_description/urdf/30cm/constants.xacro (robot description, xacro)
@@ -5,5 +5,5 @@
     Author : Theppasith N. <theppasith@gmail.com>
 -->
-<robot name="som_o_robot_20cm" xmlns:xacro="http://www.ros.org/wiki/xacro">
+<robot name="som_o_robot_30cm" xmlns:xacro="http://www.ros.org/wiki/xacro">
     <!-- Constants (m-kg-s-radians unit system) -->
     <xacro:property name="M_PI" value="3.1415926535897931"/>
@@ -15,5 +15,5 @@
     <!-- Inertial components , Mass (kgs) -->
     <xacro:property name="base_mass" value="0.2"/>
-    <xacro:property name="base_radius" value="0.20"/>
+    <xacro:property name="base_radius" value="0.30"/>
     <xacro:property name="base_height" value="0.22"/>
     <xacro:property name="base_link_visual_mesh_offset_z" value="0.55"/>
@@ -21,5 +21,5 @@
     <xacro:property name="base_col_box_height" value="0.183091"/>
     <xacro:property name="base_col_box_length" value="0.200"/>
-    <xacro:property name="base_col_box_width" value="0.130"/>
+    <xacro:property name="base_col_box_width" value="0.230"/>
     <!-- Wheels -->
     <xacro:property name="wheel_radius" value="0.042" />

File: som_o_description/urdf/30cm/som_o_robot_30cm.xacro (robot description, xacro)
@@ -7,12 +7,12 @@
 <robot name="som_o_robot_20cm" xmlns:xacro="http://www.ros.org/wiki/xacro">
   <!-- Constants -->
-  <xacro:include filename="$(find som_o_description)/urdf/20cm/constants.xacro" />
+  <xacro:include filename="$(find som_o_description)/urdf/30cm/constants.xacro" />
   <!-- Material (Color) -->
   <xacro:include filename="$(find som_o_description)/urdf/shared_components/material.xacro" />
   <!-- Body of Robot -->
       <!-- Footprint (require Base Link inclusion) -->
-      <xacro:include filename="$(find som_o_description)/urdf/20cm/base_footprint.xacro" />
+      <xacro:include filename="$(find som_o_description)/urdf/30cm/base_footprint.xacro" />
       <!-- Base Link (Main chassis) -->
-      <xacro:include filename="$(find som_o_description)/urdf/20cm/base_link.xacro" />
+      <xacro:include filename="$(find som_o_description)/urdf/30cm/base_link.xacro" />
       <!-- Wheels (Plugin) -->
       <xacro:include filename="$(find som_o_description)/urdf/shared_components/wheel.xacro" />

File: som_o_description/urdf/shared_components/diff_drive_plugin.xacro (robot description, xacro)
@@ -1,4 +1,4 @@
 <?xml version="1.0"?>
-<robot name="som_o_robot_20cm" xmlns:xacro="http://www.ros.org/wiki/xacro">
+<robot name="diff_drive_plugin" xmlns:xacro="http://www.ros.org/wiki/xacro">
     <!-- Differential drive controller  -->
     <gazebo>

File: som_o_description/urdf/shared_components/material.xacro (robot description, xacro)
@@ -1,5 +1,9 @@
 <?xml version="1.0"?>
-<robot name="som_o_robot_20cm" xmlns:xacro="http://www.ros.org/wiki/xacro">
-<!-- Definitions for colors for using in Gazebo and RViz -->
+<!--
+    Definition for colors for using in Gazebo and RViz
+    Company : Obodroid Corporation
+    Author : Theppasith N. <theppasith@gmail.com>
+-->
+<robot name="material" xmlns:xacro="http://www.ros.org/wiki/xacro">
     <material name="Black">
         <color rgba="0.0 0.0 0.0 1.0" />
